Commit message: Update finalassemblya.urdf

File: multi_robot/urdf/finalassemblya.urdf (robot description, URDF)
Before this commit: robot finalassemblya, 6 links, 5 joints
Links:
- link backleftlink: geometry collision mesh filename=package://multi_robot/meshes/backleftlink.STL; visual mesh filename=package://multi_robot/meshes/backleftlink.STL
- link backrightlink: geometry collision mesh filename=package://multi_robot/meshes/backrightlink.STL; visual mesh filename=package://multi_robot/meshes/backrightlink.STL
- link base_link: geometry collision mesh filename=package://multi_robot/meshes/base_link.STL; visual mesh filename=package://multi_robot/meshes/base_link.STL
- link frontleftlink: geometry collision mesh filename=package://multi_robot/meshes/frontleftlink.STL; visual mesh filename=package://multi_robot/meshes/frontleftlink.STL
- link frontrightlink: geometry collision mesh filename=package://multi_robot/meshes/frontrightlink.STL; visual mesh filename=package://multi_robot/meshes/frontrightlink.STL
- link moplink: geometry collision mesh filename=package://multi_robot/meshes/moplink.STL; visual mesh filename=package://multi_robot/meshes/moplink.STL
